File: Bornhack Make Tradition Badge.sch (KiCad schematic (older format))
At the start: 43 parts, among them J1 DEBUG, J2 LE UART, J3 I2C, J4 CONN_02X04, J5 CONN_02X04, J6 CONN_02X04, J7 CONN_01X02, J8 CONN_01X02, P1 USB_OTG, Q1 FDC6420C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

Commit message: Flipped D+ and D- and removed dual battery option
- D+ and D- has been corrected
- Coin cell holder has been removed, since the badge uses too much power when the screen is on for a coin cell to be a reasonable power source.
- Current measurement pin headers have also been removed.

Signed-off-by: Thomas Flummer <tf@flummer.net>
Parts:
- removed BT1: 3V Button cell, Power:Linx_BAT_HLD_001, symbol Battery_Cell
- removed J7, J8: CONN_01X02, Pin_Headers:Pin_Header_Straight_1x02_Pitch2.54mm, symbol CONN_01X02
Connections:
- net VBAT: now also BT2.1 (+)
- net at U1.35 (PC14): now also R5.2; no longer R6.2
- net at U1.36 (PC15): now also R6.2; no longer R5.2
- net at P1.2 (D-), R5.1: now also R4.1
- net at P1.3 (D+), R6.1: no longer R4.1
Changed lines of the file:
@@
 LIBS:Semiconductors
 LIBS:Bornhack Make Tradition Badge-cache
-EELAYER 26 0
+EELAYER 25 0
 EELAYER END
 $Descr A4 11693 8268
@@
 Connection ~ 6800 2500
 Wire Wire Line
-	6950 2600 6150 2600
-Wire Wire Line
-	6950 2700 6150 2700
-Wire Wire Line
-	5850 2700 5450 2700
-Wire Wire Line
-	5450 2700 5450 2800
-Wire Wire Line
-	5450 2800 4950 2800
-Wire Wire Line
 	5850 2600 5350 2600
-Wire Wire Line
-	5350 2600 5350 2700
-Wire Wire Line
-	5350 2700 4950 2700
 Wire Wire Line
 	2550 3000 1950 3000
@@
 	7050 3700 10400 3700
 Wire Wire Line
-	6200 2700 6200 2200
-Wire Wire Line
 	6200 2200 6000 2200
-Connection ~ 6200 2700
 Wire Wire Line
 	5700 2200 5300 2200
@@
 	1100 3400 1000 3400
 $Comp
-L Battery_Cell BT1
-U 1 1 596C8356
-P 6200 1400
-F 0 "BT1" H 6318 1496 50  0000 L CNN
-F 1 "3V Button cell" H 6318 1405 50  0000 L CNN
-F 2 "Power:Linx_BAT_HLD_001" V 6200 1460 50  0001 C CNN
-F 3 "" V 6200 1460 50  0001 C CNN
-	1    6200 1400
-	1    0    0    -1
-$EndComp
-$Comp
 L Battery_Cell BT2
 U 1 1 596C8411
@@
 	1    0    0    -1
 $EndComp
+Wire Wire Line
+	7200 1900 7200 2000
+Wire Wire Line
+	7200 1500 7200 1600
+Text GLabel 7350 850  2    60   Input ~ 0
+VBAT
 $Comp
 L GND #PWR027
-U 1 1 596C89CB
-P 6200 1600
-F 0 "#PWR027" H 6200 1350 50  0001 C CNN
-F 1 "GND" H 6205 1427 50  0000 C CNN
-F 2 "" H 6200 1600 50  0000 C CNN
-F 3 "" H 6200 1600 50  0000 C CNN
-	1    6200 1600
-	1    0    0    -1
-$EndComp
-Wire Wire Line
-	7200 1900 7200 2000
-Wire Wire Line
-	7200 1500 7200 1600
-Wire Wire Line
-	6200 1500 6200 1600
-$Comp
-L CONN_01X02 J7
-U 1 1 596C92E7
-P 5900 1050
-F 0 "J7" H 5819 775 50  0000 C CNN
-F 1 "CONN_01X02" H 5819 866 50  0000 C CNN
-F 2 "Pin_Headers:Pin_Header_Straight_1x02_Pitch2.54mm" H 5900 1050 50  0001 C CNN
-F 3 "" H 5900 1050 50  0001 C CNN
-	1    5900 1050
-	-1   0    0    1
-$EndComp
-$Comp
-L CONN_01X02 J8
-U 1 1 596C962B
-P 6900 1050
-F 0 "J8" H 6819 775 50  0000 C CNN
-F 1 "CONN_01X02" H 6819 866 50  0000 C CNN
-F 2 "Pin_Headers:Pin_Header_Straight_1x02_Pitch2.54mm" H 6900 1050 50  0001 C CNN
-F 3 "" H 6900 1050 50  0001 C CNN
-	1    6900 1050
-	-1   0    0    1
-$EndComp
-Wire Wire Line
-	6100 1100 6200 1100
-Wire Wire Line
-	6200 1100 6200 1200
-Wire Wire Line
-	7100 1100 7200 1100
-Wire Wire Line
-	7200 1100 7200 1200
-Text GLabel 7900 700  2    60   Input ~ 0
-VBAT
-Wire Wire Line
-	7900 700  6300 700
-Wire Wire Line
-	6300 700  6300 1000
-Wire Wire Line
-	6300 1000 6100 1000
-Wire Wire Line
-	7100 1000 7350 1000
-Wire Wire Line
-	7350 1000 7350 700
-Connection ~ 7350 700
-$Comp
-L GND #PWR028
 U 1 1 596CD5BD
 P 6850 3200
-F 0 "#PWR028" H 6850 2950 50  0001 C CNN
+F 0 "#PWR027" H 6850 2950 50  0001 C CNN
 F 1 "GND" H 6855 3027 50  0000 C CNN
 F 2 "" H 6850 3200 50  0000 C CNN
@@
 $EndComp
 $Comp
-L GND #PWR029
+L GND #PWR028
 U 1 1 596D0104
 P 800 800
-F 0 "#PWR029" H 800 550 50  0001 C CNN
+F 0 "#PWR028" H 800 550 50  0001 C CNN
 F 1 "GND" H 805 627 50  0000 C CNN
 F 2 "" H 800 800 50  0000 C CNN
@@
 $EndComp
 $Comp
-L +3.3V #PWR030
+L +3.3V #PWR029
 U 1 1 596D01AF
 P 1500 800
-F 0 "#PWR030" H 1500 650 50  0001 C CNN
+F 0 "#PWR029" H 1500 650 50  0001 C CNN
 F 1 "+3.3V" H 1515 973 50  0000 C CNN
 F 2 "" H 1500 800 50  0000 C CNN
@@
 $EndComp
 $Comp
-L GND #PWR031
+L GND #PWR030
 U 1 1 596D0801
 P 800 1550
-F 0 "#PWR031" H 800 1300 50  0001 C CNN
+F 0 "#PWR030" H 800 1300 50  0001 C CNN
 F 1 "GND" H 805 1377 50  0000 C CNN
 F 2 "" H 800 1550 50  0000 C CNN
@@
 $EndComp
 $Comp
-L +3.3V #PWR032
+L +3.3V #PWR031
 U 1 1 596D0807
 P 1500 1550
-F 0 "#PWR032" H 1500 1400 50  0001 C CNN
+F 0 "#PWR031" H 1500 1400 50  0001 C CNN
 F 1 "+3.3V" H 1515 1723 50  0000 C CNN
 F 2 "" H 1500 1550 50  0000 C CNN
@@
 $EndComp
 $Comp
-L GND #PWR033
+L GND #PWR032
 U 1 1 596D0883
 P 800 2300
-F 0 "#PWR033" H 800 2050 50  0001 C CNN
+F 0 "#PWR032" H 800 2050 50  0001 C CNN
 F 1 "GND" H 805 2127 50  0000 C CNN
 F 2 "" H 800 2300 50  0000 C CNN
@@
 $EndComp
 $Comp
-L +3.3V #PWR034
+L +3.3V #PWR033
 U 1 1 596D0889
 P 1500 2300
-F 0 "#PWR034" H 1500 2150 50  0001 C CNN
+F 0 "#PWR033" H 1500 2150 50  0001 C CNN
 F 1 "+3.3V" H 1515 2473 50  0000 C CNN
 F 2 "" H 1500 2300 50  0000 C CNN
@@
 $EndComp
 $Comp
-L GND #PWR035
+L GND #PWR034
 U 1 1 596D287C
 P 1100 4800
-F 0 "#PWR035" H 1100 4550 50  0001 C CNN
+F 0 "#PWR034" H 1100 4550 50  0001 C CNN
 F 1 "GND" H 1105 4627 50  0000 C CNN
 F 2 "" H 1100 4800 50  0000 C CNN
@@
 $EndComp
 $Comp
-L +3.3V #PWR036
+L +3.3V #PWR035
 U 1 1 596D2882
 P 1100 4300
-F 0 "#PWR036" H 1100 4150 50  0001 C CNN
+F 0 "#PWR035" H 1100 4150 50  0001 C CNN
 F 1 "+3.3V" H 1115 4473 50  0000 C CNN
 F 2 "" H 1100 4300 50  0000 C CNN
@@
 $EndComp
 $Comp
-L GND #PWR037
+L GND #PWR036
 U 1 1 596D3024
 P 1100 5800
-F 0 "#PWR037" H 1100 5550 50  0001 C CNN
+F 0 "#PWR036" H 1100 5550 50  0001 C CNN
 F 1 "GND" H 1105 5627 50  0000 C CNN
 F 2 "" H 1100 5800 50  0000 C CNN
@@
 $EndComp
 $Comp
-L +3.3V #PWR038
+L +3.3V #PWR037
 U 1 1 596D302A
 P 1100 5300
-F 0 "#PWR038" H 1100 5150 50  0001 C CNN
+F 0 "#PWR037" H 1100 5150 50  0001 C CNN
 F 1 "+3.3V" H 1115 5473 50  0000 C CNN
 F 2 "" H 1100 5300 50  0000 C CNN
@@
 Text GLabel 1200 5600 2    60   Input ~ 0
 I2C0_SDA
+Wire Wire Line
+	7350 850  7200 850
+Wire Wire Line
+	7200 850  7200 1200
+Wire Wire Line
+	6950 2700 6150 2700
+Wire Wire Line
+	6150 2600 6950 2600
+Wire Wire Line
+	6200 2200 6200 2600
+Connection ~ 6200 2600
+Wire Wire Line
+	5850 2700 4950 2700
+Wire Wire Line
+	5350 2600 5350 2800
+Wire Wire Line
+	5350 2800 4950 2800
 $EndSCHEMATC

Commit message: Changed pins for 2 buttons, cleanup and proto pads
- Changed the pins for the LEFT (X) and RIGHT (Y) buttons so that all buttons have their own interrupt
- Changed the name of the buttons to A, B, X and Y so that the names also make sense, when the badge is oriented differently
- Removed silkscreen lines around buttons and non populated pin headers
- Added SMD prototyping area on the back
- Added Open Hardware Logo and CC-BY-SA graphics
- Updated gerber files (production run)

Signed-off-by: Thomas Flummer <tf@flummer.net>
Parts:
- R2: value 1K -> 1.2K
- R3: value 1K -> 820
- SW1: value RESET -> BOOT
- SW3: value UP -> A
- SW4: value DOWN -> B
- SW5: value RIGHT -> Y
- SW6: value LEFT -> X
Connections:
- net DOWN renamed BUTTON_B
- net LEFT renamed BUTTON_X
- net BUTTON_X: now also U1.46 (PE11); no longer U1.42 (PF5)
- net PE10 renamed BUTTON_Y
- net BUTTON_Y: now also SW5.2; no longer J5.7 (P7)
- net PE11 renamed PF4
- net PF4: now also U1.41 (PF4); no longer U1.46 (PE11)
- removed net RIGHT: SW5.2, U1.41 (PF4)
- net UP renamed BUTTON_A
- new net PF5: J5.7 (P7), U1.42 (PF5)
Other:
- moved on the sheet: SW3, SW4
Changed lines of the file:
@@
 LIBS:Semiconductors
 LIBS:Bornhack Make Tradition Badge-cache
-EELAYER 25 0
+EELAYER 26 0
 EELAYER END
 $Descr A4 11693 8268
@@
 P 1700 6600
 F 0 "SW1" H 1700 6855 50  0000 C CNN
-F 1 "RESET" H 1700 6764 50  0000 C CNN
+F 1 "BOOT" H 1700 6764 50  0000 C CNN
 F 2 "Buttons_Switches_SMD:SW_SPST_PTS645" H 1700 6600 50  0001 C CNN
 F 3 "" H 1700 6600 50  0000 C CNN
@@
 P 5200 6550
 F 0 "SW5" H 5200 6805 50  0000 C CNN
-F 1 "RIGHT" H 5200 6714 50  0000 C CNN
+F 1 "Y" H 5200 6714 50  0000 C CNN
 F 2 "Buttons_Switches_SMD:SW_SPST_PTS645" H 5200 6550 50  0001 C CNN
 F 3 "" H 5200 6550 50  0000 C CNN
@@
 L SW_PUSH SW4
 U 1 1 59641C7E
-P 3875 7150
-F 0 "SW4" H 3875 7405 50  0000 C CNN
-F 1 "DOWN" H 3875 7314 50  0000 C CNN
-F 2 "Buttons_Switches_SMD:SW_SPST_PTS645" H 3875 7150 50  0001 C CNN
-F 3 "" H 3875 7150 50  0000 C CNN
-	1    3875 7150
+P 3575 7150
+F 0 "SW4" H 3575 7405 50  0000 C CNN
+F 1 "B" H 3575 7314 50  0000 C CNN
+F 2 "Buttons_Switches_SMD:SW_SPST_PTS645" H 3575 7150 50  0001 C CNN
+F 3 "" H 3575 7150 50  0000 C CNN
+	1    3575 7150
 	1    0    0    -1
 $EndComp
@@
 L SW_PUSH SW3
 U 1 1 59641CCA
-P 3875 6550
-F 0 "SW3" H 3875 6805 50  0000 C CNN
-F 1 "UP" H 3875 6714 50  0000 C CNN
-F 2 "Buttons_Switches_SMD:SW_SPST_PTS645" H 3875 6550 50  0001 C CNN
-F 3 "" H 3875 6550 50  0000 C CNN
-	1    3875 6550
+P 3575 6550
+F 0 "SW3" H 3575 6805 50  0000 C CNN
+F 1 "A" H 3575 6714 50  0000 C CNN
+F 2 "Buttons_Switches_SMD:SW_SPST_PTS645" H 3575 6550 50  0001 C CNN
+F 3 "" H 3575 6550 50  0000 C CNN
+	1    3575 6550
 	1    0    0    -1
 $EndComp
@@
 P 5200 7150
 F 0 "SW6" H 5200 7405 50  0000 C CNN
-F 1 "LEFT" H 5200 7314 50  0000 C CNN
+F 1 "X" H 5200 7314 50  0000 C CNN
 F 2 "Buttons_Switches_SMD:SW_SPST_PTS645" H 5200 7150 50  0001 C CNN
 F 3 "" H 5200 7150 50  0000 C CNN
@@
 L GND #PWR015
 U 1 1 59641FCD
-P 3525 6600
-F 0 "#PWR015" H 3525 6350 50  0001 C CNN
-F 1 "GND" H 3530 6427 50  0000 C CNN
-F 2 "" H 3525 6600 50  0000 C CNN
-F 3 "" H 3525 6600 50  0000 C CNN
-	1    3525 6600
+P 3225 6600
+F 0 "#PWR015" H 3225 6350 50  0001 C CNN
+F 1 "GND" H 3230 6427 50  0000 C CNN
+F 2 "" H 3225 6600 50  0000 C CNN
+F 3 "" H 3225 6600 50  0000 C CNN
+	1    3225 6600
 	1    0    0    -1
 $EndComp
@@
 L GND #PWR017
 U 1 1 596421DB
-P 3525 7200
-F 0 "#PWR017" H 3525 6950 50  0001 C CNN
-F 1 "GND" H 3530 7027 50  0000 C CNN
-F 2 "" H 3525 7200 50  0000 C CNN
-F 3 "" H 3525 7200 50  0000 C CNN
-	1    3525 7200
+P 3225 7200
+F 0 "#PWR017" H 3225 6950 50  0001 C CNN
+F 1 "GND" H 3230 7027 50  0000 C CNN
+F 2 "" H 3225 7200 50  0000 C CNN
+F 3 "" H 3225 7200 50  0000 C CNN
+	1    3225 7200
 	1    0    0    -1
 $EndComp
@@
 	1    0    0    -1
 $EndComp
-Text GLabel 4275 6550 2    60   Input ~ 0
-UP
-Text GLabel 4275 7150 2    60   Input ~ 0
-DOWN
+Text GLabel 3975 6550 2    60   Input ~ 0
+BUTTON_A
+Text GLabel 3975 7150 2    60   Input ~ 0
+BUTTON_B
 Text GLabel 5600 6550 2    60   Input ~ 0
-RIGHT
+BUTTON_Y
 Text GLabel 5600 7150 2    60   Input ~ 0
-LEFT
+BUTTON_X
 $Comp
 L SSD1306 OLEDM1
@@
 U 1 1 59647C36
 P 9650 3950
-F 0 "R9" H 9720 3996 50  0000 L CNN
-F 1 "10K" H 9720 3905 50  0000 L CNN
+F 0 "R9" H 9500 4000 50  0000 L CNN
+F 1 "10K" H 9450 3900 50  0000 L CNN
 F 2 "Resistors_SMD:R_0805" V 9580 3950 50  0001 C CNN
 F 3 "" H 9650 3950 50  0000 C CNN
@@
 P 3800 5800
 F 0 "R2" V 3700 5800 50  0000 C CNN
-F 1 "1K" V 3800 5800 50  0000 C CNN
+F 1 "1.2K" V 3800 5800 50  0000 C CNN
 F 2 "Resistors_SMD:R_0805" V 3730 5800 50  0001 C CNN
 F 3 "" H 3800 5800 50  0000 C CNN
@@
 P 3800 6000
 F 0 "R3" V 3700 6000 50  0000 C CNN
-F 1 "1K" V 3800 6000 50  0000 C CNN
+F 1 "820" V 3800 6000 50  0000 C CNN
 F 2 "Resistors_SMD:R_0805" V 3730 6000 50  0001 C CNN
 F 3 "" H 3800 6000 50  0000 C CNN
@@
 	4850 7150 4850 7200
 Wire Wire Line
-	3575 7150 3525 7150
-Wire Wire Line
-	3525 7150 3525 7200
-Wire Wire Line
-	3575 6550 3525 6550
-Wire Wire Line
-	3525 6550 3525 6600
+	3275 7150 3225 7150
+Wire Wire Line
+	3225 7150 3225 7200
+Wire Wire Line
+	3275 6550 3225 6550
+Wire Wire Line
+	3225 6550 3225 6600
 Wire Wire Line
 	5600 6550 5500 6550
@@
 	5600 7150 5500 7150
 Wire Wire Line
-	4275 7150 4175 7150
-Wire Wire Line
-	4275 6550 4175 6550
+	3975 7150 3875 7150
+Wire Wire Line
+	3975 6550 3875 6550
 Wire Wire Line
 	9500 5700 9850 5700
@@
 	3400 4550 3400 4450
 Text GLabel 4100 1950 1    60   Input ~ 0
-UP
+BUTTON_A
 Text GLabel 4000 1950 1    60   Input ~ 0
-DOWN
-Text GLabel 3900 1950 1    60   Input ~ 0
-RIGHT
-Text GLabel 3800 1950 1    60   Input ~ 0
-LEFT
-Wire Wire Line
-	3800 1950 3800 2050
-Wire Wire Line
-	3900 1950 3900 2050
+BUTTON_B
+Text GLabel 3500 1950 1    60   Input ~ 0
+BUTTON_Y
+Text GLabel 3400 1950 1    60   Input ~ 0
+BUTTON_X
 Wire Wire Line
 	4000 1950 4000 2050
@@
 Text GLabel 4950 3100 2    60   Input ~ 0
 PC10
-Text GLabel 3500 2050 1    60   Input ~ 0
-PE10
-Text GLabel 3400 2050 1    60   Input ~ 0
-PE11
 $Comp
 L CONN_02X04 J4
@@
 Text GLabel 1400 1850 2    60   Input ~ 0
 PD7
-Text GLabel 900  1950 0    60   Input ~ 0
-PE10
-Text GLabel 1400 1950 2    60   Input ~ 0
-PE11
 Text GLabel 900  2500 0    60   Input ~ 0
 PB11
@@
 Wire Wire Line
 	5350 2800 4950 2800
+Wire Wire Line
+	3400 1950 3400 2050
+Wire Wire Line
+	3500 1950 3500 2050
+Text GLabel 3800 2050 1    60   Input ~ 0
+PF5
+Text GLabel 3900 2050 1    60   Input ~ 0
+PF4
+Text GLabel 900  1950 0    60   Input ~ 0
+PF5
+Text GLabel 1400 1950 2    60   Input ~ 0
+PF4
 $EndSCHEMATC
